File: NEW PSU.kicad_pcb (KiCad board)
At the start: 2 copper layers, 181.5 x 95.5 mm, 21 parts, among them J1 12v +, J2 12 v -, J3 5v, J4 Conn_01x01_Socket, J5 Conn_01x01_Socket, U1 L7812, U2 L7912, U3 L7805

Commit message: Add files via upload
Parts:
- added J6: Conn_01x01_Socket, Connector_Wago:Wago_734-132_1x02_P3.50mm_Vertical, F.Cu at (179.2, 72.8)
- C1: value 1000uF\35v -> 2200uF\35v
- C2: value 1000uf\50v -> 2200uf\50v
- moved C11 94.7 mm to (157.2, 48.9), turned to -90 degrees
- moved C12 82.0 mm to (180.0, 54.2), turned to -90 degrees
- moved C6 64.5 mm to (152.4, 120.8), turned to 180 degrees
- moved C8 57.0 mm to (175.0, 105.0)
- moved C10 56.8 mm to (105.8, 50.8), turned to -90 degrees
- moved C2 53.6 mm to (80.5, 112.0), turned to -90 degrees
- moved C4 44.9 mm to (98.8, 100.2), turned to -90 degrees
- moved C3 41.8 mm to (101.2, 79.0), turned to -90 degrees
- moved J3 40.4 mm to (196.5, 46.2)
- moved C7 39.7 mm to (138.2, 93.2), turned to 90 degrees
- moved C9 36.9 mm to (80.4, 54.0)
- moved U3 36.0 mm to (126.1, 44.2)
- moved U1 34.8 mm to (114.7, 81.2)
- moved U2 25.2 mm to (109.2, 122.2), turned to -90 degrees
- moved C5 23.1 mm to (127.8, 80.3), turned to 90 degrees
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- renumbered J5 to J1, J4 to J2, J1 to J4, J2 to J5
Routing:
- net GND: track 0.00 -> 481.0 mm
- net Net-(D1-+): track 0.00 -> 123.4 mm
- net Net-(J4-Pin_1): track 0.00 -> 107.9 mm
- net Net-(J5-Pin_1): track 0.00 -> 107.7 mm, vias 0 -> 1
- net Net-(D1--): track 0.00 -> 98.1 mm
- net Net-(J3-Pin_1): track 0.00 -> 88.2 mm
- net Net-(J1-Pin_1): track 0.00 -> 29.0 mm
- net Net-(J2-Pin_1): track 0.00 -> 16.8 mm
- added copper zone on B.Cu, net GND
Other:
- board size 181.5 x 95.5 mm -> 181.5 x 93 mm

Commit message: Add files via upload
Parts:
- removed J3: 5v, Connector_Wago:Wago_734-132_1x02_P3.50mm_Vertical
- removed J4: 12v +, Connector_Wago:Wago_734-132_1x02_P3.50mm_Vertical
- removed J5: 12 v -, Connector_Wago:Wago_734-132_1x02_P3.50mm_Vertical
- removed J6: Conn_01x01_Socket, Connector_Wago:Wago_734-132_1x02_P3.50mm_Vertical
- added J7: Conn_01x04, Connector_FFC-FPC:Hirose_FH41-30S-0.5SH_1x30_1MP_1SH_P0.5mm_Horizontal, F.Cu at (205.8, 59.0)
- U1: footprint Package_TO_SOT_SMD:TO-252-2 -> Package_TO_SOT_THT:TO-220-3_Vertical
- U2: footprint Package_TO_SOT_SMD:TO-263-2 -> Package_TO_SOT_THT:TO-220-3_Vertical
- moved C9 7.29 mm to (78.8, 46.9), turned to -90 degrees
- moved U1 6.49 mm to (113.0, 75.0)
- moved C6 2.76 mm to (154.0, 118.5), turned to -90 degrees
- turned J1 to -90 degrees
- turned J2 to -90 degrees
- turned U2 to 180 degrees
Routing:
- net GND: track 481.0 -> 401.1 mm
- net Net-(J7-Pin_4): track 107.7 -> 125.9 mm, vias 1 -> 0
- net Net-(D1-+): track 123.4 -> 138.4 mm
- net Net-(J7-Pin_3): track 107.9 -> 95.3 mm, vias 0 -> 1
- net Net-(D1--): track 98.1 -> 101.1 mm
- net Net-(J7-Pin_2): track 88.2 -> 85.7 mm
- removed copper zone on B.Cu, net GND

Commit message: Add files via upload
Parts:
- removed J7: Conn_01x04, Connector_FFC-FPC:Hirose_FH41-30S-0.5SH_1x30_1MP_1SH_P0.5mm_Horizontal
- added D2: LED, LED_THT:LED_D1.8mm_W1.8mm_H2.4mm_Horizontal_O1.27mm_Z1.6mm, F.Cu at (184.0, 61.5)
- added D3: LED, LED_THT:LED_D1.8mm_W1.8mm_H2.4mm_Horizontal_O1.27mm_Z1.6mm, F.Cu at (173.8, 94.4)
- added D4: LED, LED_THT:LED_D1.8mm_W1.8mm_H2.4mm_Horizontal_O1.27mm_Z1.6mm, F.Cu at (167.0, 119.9)
- added J3: Conn_01x01_Socket, Connector:JWT_A3963_1x02_P3.96mm_Vertical, F.Cu at (127.3, 44.0)
- added J4: Conn_01x04, Connector_Molex:Molex_KK-396_A-41791-0004_1x04_P3.96mm_Vertical, F.Cu at (217.5, 83.0)
- added R1: 2000, Resistor_THT:R_Axial_DIN0309_L9.0mm_D3.2mm_P15.24mm_Horizontal, F.Cu at (183.9, 64.9)
- added R2: 2000, Resistor_THT:R_Axial_DIN0309_L9.0mm_D3.2mm_P15.24mm_Horizontal, F.Cu at (180.9, 89.2)
- added R3: 2000, Resistor_THT:R_Axial_DIN0309_L9.0mm_D3.2mm_P15.24mm_Horizontal, F.Cu at (179.5, 102.6)
- moved C6 27.5 mm to (126.5, 119.2)
- moved C8 27.5 mm to (147.5, 105.8)
- moved C12 21.1 mm to (171.2, 73.5)
- moved C11 17.4 mm to (158.4, 66.2), turned to 180 degrees
- moved U3 10.8 mm to (127.0, 55.0)
- moved C5 9.52 mm to (125.5, 89.5)
- moved C9 3.14 mm to (80.8, 49.2)
Routing:
- net Net-(D2-A): track 85.7 -> 129.7 mm
- net Net-(D3-A): track 95.3 -> 133.2 mm, vias 1 -> 0
- net Net-(D4-A): track 125.9 -> 158.6 mm
- net GND: track 401.1 -> 422.8 mm
- net Net-(D4-K): track 0.00 -> 13.3 mm
- net Net-(D3-K): track 0.00 -> 9.26 mm
- net Net-(D2-K): track 0.00 -> 3.43 mm
- net Net-(D1-+): track 138.4 -> 137.6 mm
- added copper zone on B.Cu, net GND
Other:
- board size 181.5 x 93 mm -> 188.2 x 93 mm
- rule pad_to_mask_clearance: 0.02 -> 0
